File: uCLUCE_PCB.sch (KiCad schematic (older format))
At the start: 3 parts, among them P1 USB_A, U1 PIC16F1455-I/ST, U2 MCP2003B

Commit message: Coponents add
Parts:
- added C1: 0.47u, Capacitors_SMD:C_0603, symbol C_Small
- added C2, C3: 100n, Capacitors_SMD:C_0603, symbol C_Small
- added D1: D, Diodes_SMD:D_0805, symbol D
- added ICS1: Conn_01x05, Pin_Headers:Pin_Header_Straight_1x05_Pitch2.54mm, symbol Conn_01x05
- added J1: Screw_Terminal_01x03, Connectors:AK300-3, symbol Screw_Terminal_01x03
- added J2: GS2, Connectors:GS2, symbol GS2
- added R1: 1k, Resistors_SMD:R_0603, symbol R_Small
- P1: symbol USB_A -> USB_A-RESCUE-uCLUCE_PCB
Connections:
- net labels added: +5V, +BATT, GND, MCLR
- wire segments 0 -> 25
Other:
- moved on the sheet: U2

Commit message: Route
Parts:
- added C4: 220p, Capacitors_SMD:C_0603, symbol C_Small
- added C5: 1u, Capacitors_SMD:C_0603, symbol C_Small
- added R2: 4,7k, Resistors_SMD:R_0603, symbol R_Small
- C2: value 100n -> 470n
Connections:
- net +5V: now also R2.2
- net +BATT: now also C5.2
- net GND: now also C4.1, C5.1
- net at U1.6 (RC4), U2.1 (Rxd): now also R2.1
- net at J1.2 (Pin_2), J2.2 (G2), U2.6 (LBB): now also C4.2
Changed lines of the file:
@@
 EESchema Schematic File Version 2
-LIBS:uCLUCE_PCB-rescue
 LIBS:power
 LIBS:device
@@
 $EndComp
 $Comp
-L GND #PWR9
+L GND #PWR13
 U 1 1 59E21F8A
 P 4550 2300
-F 0 "#PWR9" H 4550 2050 50  0001 C CNN
+F 0 "#PWR13" H 4550 2050 50  0001 C CNN
 F 1 "GND" H 4550 2150 50  0001 C CNN
 F 2 "" H 4550 2300 50  0001 C CNN
@@
 $EndComp
 $Comp
-L GND #PWR11
+L GND #PWR15
 U 1 1 59E21FB8
 P 5350 1800
-F 0 "#PWR11" H 5350 1550 50  0001 C CNN
+F 0 "#PWR15" H 5350 1550 50  0001 C CNN
 F 1 "GND" H 5350 1650 50  0000 C CNN
 F 2 "" H 5350 1800 50  0001 C CNN
@@
 $EndComp
 $Comp
-L +5V #PWR13
+L +5V #PWR17
 U 1 1 59E220C9
 P 5350 2900
-F 0 "#PWR13" H 5350 2750 50  0001 C CNN
+F 0 "#PWR17" H 5350 2750 50  0001 C CNN
 F 1 "+5V" H 5350 3040 50  0000 C CNN
 F 2 "" H 5350 2900 50  0001 C CNN
@@
 $EndComp
 $Comp
-L +5V #PWR8
+L +5V #PWR11
 U 1 1 59E2213F
 P 2450 2000
-F 0 "#PWR8" H 2450 1850 50  0001 C CNN
+F 0 "#PWR11" H 2450 1850 50  0001 C CNN
 F 1 "+5V" H 2450 2140 50  0000 C CNN
 F 2 "" H 2450 2000 50  0001 C CNN
@@
 $EndComp
 $Comp
-L +BATT #PWR2
+L +BATT #PWR1
 U 1 1 59E22154
-P 900 2600
-F 0 "#PWR2" H 900 2450 50  0001 C CNN
-F 1 "+BATT" H 900 2740 50  0000 C CNN
-F 2 "" H 900 2600 50  0001 C CNN
-F 3 "" H 900 2600 50  0001 C CNN
-	1    900  2600
-	-1   0    0    1
-$EndComp
-$Comp
-L GND #PWR1
+P 750 2800
+F 0 "#PWR1" H 750 2650 50  0001 C CNN
+F 1 "+BATT" H 750 2940 50  0000 C CNN
+F 2 "" H 750 2800 50  0001 C CNN
+F 3 "" H 750 2800 50  0001 C CNN
+	1    750  2800
+	1    0    0    -1
+$EndComp
+$Comp
+L GND #PWR2
 U 1 1 59E22180
-P 900 2400
-F 0 "#PWR1" H 900 2150 50  0001 C CNN
-F 1 "GND" H 900 2250 50  0000 C CNN
-F 2 "" H 900 2400 50  0001 C CNN
-F 3 "" H 900 2400 50  0001 C CNN
-	1    900  2400
-	-1   0    0    1
+P 800 2200
+F 0 "#PWR2" H 800 1950 50  0001 C CNN
+F 1 "GND" H 800 2050 50  0000 C CNN
+F 2 "" H 800 2200 50  0001 C CNN
+F 3 "" H 800 2200 50  0001 C CNN
+	1    800  2200
+	1    0    0    -1
 $EndComp
 $Comp
@@
 $EndComp
 $Comp
-L GND #PWR12
+L GND #PWR16
 U 1 1 59E230A7
 P 5350 2800
-F 0 "#PWR12" H 5350 2550 50  0001 C CNN
+F 0 "#PWR16" H 5350 2550 50  0001 C CNN
 F 1 "GND" V 5300 2600 50  0001 C CNN
 F 2 "" H 5350 2800 50  0001 C CNN
@@
 MCLR
 $Comp
-L +5V #PWR10
+L +5V #PWR14
 U 1 1 59E237FB
 P 4950 2300
-F 0 "#PWR10" H 4950 2150 50  0001 C CNN
+F 0 "#PWR14" H 4950 2150 50  0001 C CNN
 F 1 "+5V" H 4950 2440 50  0000 C CNN
 F 2 "" H 4950 2300 50  0001 C CNN
@@
 P 1850 1850
 F 0 "C2" H 1950 1850 50  0000 L CNN
-F 1 "100n" H 1900 1950 50  0000 L CNN
+F 1 "470n" H 1900 1950 50  0000 L CNN
 F 2 "Capacitors_SMD:C_0603" H 1850 1850 50  0001 C CNN
 F 3 "" H 1850 1850 50  0001 C CNN
@@
 $EndComp
 $Comp
-L +5V #PWR4
+L +5V #PWR7
 U 1 1 59E2335A
 P 1850 1750
-F 0 "#PWR4" H 1850 1600 50  0001 C CNN
+F 0 "#PWR7" H 1850 1600 50  0001 C CNN
 F 1 "+5V" H 1850 1890 50  0000 C CNN
 F 2 "" H 1850 1750 50  0001 C CNN
@@
 $EndComp
 $Comp
-L GND #PWR5
+L GND #PWR8
 U 1 1 59E2337A
 P 1850 1950
-F 0 "#PWR5" H 1850 1700 50  0001 C CNN
+F 0 "#PWR8" H 1850 1700 50  0001 C CNN
 F 1 "GND" H 1850 1800 50  0001 C CNN
 F 2 "" H 1850 1950 50  0001 C CNN
@@
 $EndComp
 $Comp
-L +5V #PWR6
+L +5V #PWR9
 U 1 1 59E233BF
 P 2150 1750
-F 0 "#PWR6" H 2150 1600 50  0001 C CNN
+F 0 "#PWR9" H 2150 1600 50  0001 C CNN
 F 1 "+5V" H 2150 1890 50  0000 C CNN
 F 2 "" H 2150 1750 50  0001 C CNN
@@
 $EndComp
 $Comp
-L GND #PWR7
+L GND #PWR10
 U 1 1 59E23423
 P 2150 1950
-F 0 "#PWR7" H 2150 1700 50  0001 C CNN
+F 0 "#PWR10" H 2150 1700 50  0001 C CNN
 F 1 "GND" H 2150 1800 50  0001 C CNN
 F 2 "" H 2150 1950 50  0001 C CNN
@@
 Wire Wire Line
 	1100 2600 750  2600
-Connection ~ 900  2600
+Connection ~ 800  2600
 Wire Wire Line
 	750  2500 1100 2500
@@
 Connection ~ 1050 2500
 $Comp
-L +BATT #PWR3
+L +BATT #PWR4
 U 1 1 59E23A89
 P 1050 1600
-F 0 "#PWR3" H 1050 1450 50  0001 C CNN
+F 0 "#PWR4" H 1050 1450 50  0001 C CNN
 F 1 "+BATT" H 1050 1740 50  0000 C CNN
 F 2 "" H 1050 1600 50  0001 C CNN
@@
 	-1   0    0    1
 $EndComp
+$Comp
+L C_Small C4
+U 1 1 59E5022E
+P 1000 2900
+F 0 "C4" H 1050 2850 50  0000 L CNN
+F 1 "220p" H 1050 2950 50  0000 L CNN
+F 2 "Capacitors_SMD:C_0603" H 1000 2900 50  0001 C CNN
+F 3 "" H 1000 2900 50  0001 C CNN
+	1    1000 2900
+	-1   0    0    1
+$EndComp
+Wire Wire Line
+	1000 2800 1000 2500
+Connection ~ 1000 2500
+$Comp
+L GND #PWR3
+U 1 1 59E50704
+P 1000 3000
+F 0 "#PWR3" H 1000 2750 50  0001 C CNN
+F 1 "GND" H 1000 2850 50  0000 C CNN
+F 2 "" H 1000 3000 50  0001 C CNN
+F 3 "" H 1000 3000 50  0001 C CNN
+	1    1000 3000
+	1    0    0    -1
+$EndComp
+$Comp
+L R_Small R2
+U 1 1 59E50B0E
+P 2350 2600
+F 0 "R2" H 2400 2650 50  0000 L CNN
+F 1 "4,7k" H 2400 2550 50  0000 L CNN
+F 2 "Resistors_SMD:R_0603" H 2350 2600 50  0001 C CNN
+F 3 "" H 2350 2600 50  0001 C CNN
+	1    2350 2600
+	1    0    0    -1
+$EndComp
+Connection ~ 2350 2500
+$Comp
+L +5V #PWR12
+U 1 1 59E50C40
+P 2550 2950
+F 0 "#PWR12" H 2550 2800 50  0001 C CNN
+F 1 "+5V" H 2550 3090 50  0000 C CNN
+F 2 "" H 2550 2950 50  0001 C CNN
+F 3 "" H 2550 2950 50  0001 C CNN
+	1    2550 2950
+	1    0    0    -1
+$EndComp
+Wire Wire Line
+	2550 2950 2350 2950
+Wire Wire Line
+	2350 2950 2350 2700
+Wire Wire Line
+	900  2400 900  2200
+Wire Wire Line
+	900  2200 800  2200
+Wire Wire Line
+	750  2800 800  2800
+Wire Wire Line
+	800  2800 800  2600
+$Comp
+L C_Small C5
+U 1 1 59E51390
+P 1500 1850
+F 0 "C5" H 1600 1850 50  0000 L CNN
+F 1 "1u" H 1550 1950 50  0000 L CNN
+F 2 "Capacitors_SMD:C_0603" H 1500 1850 50  0001 C CNN
+F 3 "" H 1500 1850 50  0001 C CNN
+	1    1500 1850
+	-1   0    0    1
+$EndComp
+$Comp
+L GND #PWR6
+U 1 1 59E51428
+P 1500 1950
+F 0 "#PWR6" H 1500 1700 50  0001 C CNN
+F 1 "GND" H 1500 1800 50  0001 C CNN
+F 2 "" H 1500 1950 50  0001 C CNN
+F 3 "" H 1500 1950 50  0001 C CNN
+	1    1500 1950
+	1    0    0    -1
+$EndComp
+$Comp
+L +BATT #PWR?
+U 1 1 59E51598
+P 1500 1750
+F 0 "#PWR?" H 1500 1600 50  0001 C CNN
+F 1 "+BATT" H 1500 1890 50  0000 C CNN
+F 2 "" H 1500 1750 50  0001 C CNN
+F 3 "" H 1500 1750 50  0001 C CNN
+	1    1500 1750
+	1    0    0    -1
+$EndComp
 $EndSCHEMATC

Commit message: diodes add
Parts:
- removed C4: 220p, Capacitors_SMD:C_0603, symbol C_Small
- removed C5: 1u, Capacitors_SMD:C_0603, symbol C_Small
- added C4: 220p, symbol CP1_Small
- added C5: 1u, symbol CP1_Small
- added D2: D_Schottky_Small, Diodes_SMD:D_SMA, symbol D_Schottky_Small
- added D3: SMBD914E6327HTSA1, Diodes_SMD:D_SOT-23_ANK, symbol D
- added R3: 50, Resistors_SMD:R_0603, symbol R_Small
- D1: value D -> SMBD914E6327HTSA1; footprint Diodes_SMD:D_0805 -> Diodes_SMD:D_SOT-23_ANK; 1st Disrtib Link (none) -> https://www.tme.eu/pl/details/smbd914e6327htsa1/diody-uniwe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
- U1: 1st Disrtib Link (none) -> https://octopart.com/search?q=PIC16F1455-I%2FST
- U2: 1st Disrtib Link (none) -> https://octopart.com/search?q=MCP2003B
Connections:
- net +BATT: now also D3.2 (A); no longer U2.7 (Vbb)
- net GND: now also C4.2, C5.2, D2.2 (A)
- net at J1.2 (Pin_2), J2.2 (G2), U2.6 (LBB): now also C4.1
- new net: C5.1, D2.1 (K), R3.1, U2.7 (Vbb)
- new net: D3.1 (K), R3.2
Other:
- moved on the sheet: C1, C2, C3, ICS1, J1, J2, P1, R1, R2, U1, U2

Commit message: Footprint update
Parts:
- added P2: UART_TTL, Pin_Headers:Pin_Header_Straight_1x02_Pitch2.54mm, symbol CONN_01X02
- added U3: fiducial, Fiducials:Fiducial_1mm_Dia_2.54mm_Outer_CopperBottom, symbol fiducial
- J1: 1st Disrtib Link (none) -> https://www.maritex.com.pl/zlacza/listwy_zaciskowe/listwy_z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
- P1: footprint Connect:USB_A -> uCLUCE_PCB:USB_A_DS1097; 1st Disrtib Link (none) -> https://www.maritex.com.pl/zlacza/zlacza_usb_hdmi_ieee/zlac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
Connections:
- net at R2.1, U1.6 (RC4), U2.1 (Rxd): now also P2.2 (P2)
- net at U1.5 (RC5), U2.4 (TXd): now also P2.1 (P1)
Changed lines of the file:
@@
 LIBS:LINlib
 LIBS:PIC16F
+LIBS:custom
 LIBS:uCLUCE_PCB-cache
 EELAYER 25 0
@@
 F 0 "P1" V 7100 2000 50  0000 C CNN
 F 1 "USB_A" H 6800 2300 50  0000 C CNN
-F 2 "Connect:USB_A" V 6800 2000 50  0001 C CNN
+F 2 "uCLUCE_PCB:USB_A_DS1097" V 6800 2000 50  0001 C CNN
 F 3 "" V 6800 2000 50  0000 C CNN
+F 4 "https://www.maritex.com.pl/zlacza/zlacza_usb_hdmi_ieee/zlacza_i_kable_usb/wtyk_usb_1xa4_katowy/usbp1arw-cv.html" H 6850 2100 60  0001 C CNN "1st Disrtib Link"
 	1    6850 2100
 	0    1    -1   0
@@
 $EndComp
 $Comp
-L GND #PWR01
+L GND #PWR16
 U 1 1 59E21FB8
 P 7350 2150
-F 0 "#PWR01" H 7350 1900 50  0001 C CNN
+F 0 "#PWR16" H 7350 1900 50  0001 C CNN
 F 1 "GND" H 7350 2000 50  0000 C CNN
 F 2 "" H 7350 2150 50  0001 C CNN
@@
 $EndComp
 $Comp
-L +5V #PWR02
+L +5V #PWR15
 U 1 1 59E220C9
 P 6950 2900
-F 0 "#PWR02" H 6950 2750 50  0001 C CNN
+F 0 "#PWR15" H 6950 2750 50  0001 C CNN
 F 1 "+5V" H 6950 3040 50  0000 C CNN
 F 2 "" H 6950 2900 50  0001 C CNN
@@
 $EndComp
 $Comp
-L +5V #PWR03
+L +5V #PWR11
 U 1 1 59E2213F
 P 4050 2000
-F 0 "#PWR03" H 4050 1850 50  0001 C CNN
+F 0 "#PWR11" H 4050 1850 50  0001 C CNN
 F 1 "+5V" H 4050 2140 50  0000 C CNN
 F 2 "" H 4050 2000 50  0001 C CNN
@@
 $EndComp
 $Comp
-L +BATT #PWR04
+L +BATT #PWR1
 U 1 1 59E22154
 P 2000 2200
-F 0 "#PWR04" H 2000 2050 50  0001 C CNN
+F 0 "#PWR1" H 2000 2050 50  0001 C CNN
 F 1 "+BATT" V 1950 2400 50  0000 C CNN
 F 2 "" H 2000 2200 50  0001 C CNN
@@
 $EndComp
 $Comp
-L GND #PWR05
+L GND #PWR2
 U 1 1 59E22180
 P 2400 2200
-F 0 "#PWR05" H 2400 1950 50  0001 C CNN
+F 0 "#PWR2" H 2400 1950 50  0001 C CNN
 F 1 "GND" V 2300 2100 50  0000 C CNN
 F 2 "" H 2400 2200 50  0001 C CNN
@@
 F 2 "Connectors:AK300-3" H 1700 2500 50  0001 C CNN
 F 3 "" H 1700 2500 50  0001 C CNN
+F 4 "https://www.maritex.com.pl/zlacza/listwy_zaciskowe/listwy_zaciskowe_standard_nierozlaczalne/listwy_zaciskowe_pionowe_z_okraglym_otworem_w_rastrze_5_00mm/tbo5003s-1bk.html" H 1700 2500 60  0001 C CNN "1st Disrtib Link"
 	1    1700 2500
 	-1   0    0    1
@@
 $EndComp
 $Comp
-L GND #PWR06
+L GND #PWR14
 U 1 1 59E230A7
 P 6950 2800
-F 0 "#PWR06" H 6950 2550 50  0001 C CNN
+F 0 "#PWR14" H 6950 2550 50  0001 C CNN
 F 1 "GND" V 6900 2600 50  0001 C CNN
 F 2 "" H 6950 2800 50  0001 C CNN
@@
 MCLR
 $Comp
-L +5V #PWR07
+L +5V #PWR13
 U 1 1 59E237FB
 P 6550 2300
-F 0 "#PWR07" H 6550 2150 50  0001 C CNN
+F 0 "#PWR13" H 6550 2150 50  0001 C CNN
 F 1 "+5V" H 6550 2440 50  0000 C CNN
 F 2 "" H 6550 2300 50  0001 C CNN
@@
 $EndComp
 $Comp
-L +5V #PWR08
+L +5V #PWR7
 U 1 1 59E2335A
 P 3450 1750
-F 0 "#PWR08" H 3450 1600 50  0001 C CNN
+F 0 "#PWR7" H 3450 1600 50  0001 C CNN
 F 1 "+5V" H 3450 1890 50  0000 C CNN
 F 2 "" H 3450 1750 50  0001 C CNN
@@
 $EndComp
 $Comp
-L GND #PWR09
+L GND #PWR8
 U 1 1 59E2337A
 P 3450 1950
-F 0 "#PWR09" H 3450 1700 50  0001 C CNN
+F 0 "#PWR8" H 3450 1700 50  0001 C CNN
 F 1 "GND" H 3450 1800 50  0001 C CNN
 F 2 "" H 3450 1950 50  0001 C CNN
@@
 $EndComp
 $Comp
-L +5V #PWR010
+L +5V #PWR9
 U 1 1 59E233BF
 P 3750 1750
-F 0 "#PWR010" H 3750 1600 50  0001 C CNN
+F 0 "#PWR9" H 3750 1600 50  0001 C CNN
 F 1 "+5V" H 3750 1890 50  0000 C CNN
 F 2 "" H 3750 1750 50  0001 C CNN
@@
 $EndComp
 $Comp
-L GND #PWR011
+L GND #PWR10
 U 1 1 59E23423
 P 3750 1950
-F 0 "#PWR011" H 3750 1700 50  0001 C CNN
+F 0 "#PWR10" H 3750 1700 50  0001 C CNN
 F 1 "GND" H 3750 1800 50  0001 C CNN
 F 2 "" H 3750 1950 50  0001 C CNN
@@
 $EndComp
 $Comp
-L +BATT #PWR012
+L +BATT #PWR3
 U 1 1 59E23A89
 P 2650 1050
-F 0 "#PWR012" H 2650 900 50  0001 C CNN
+F 0 "#PWR3" H 2650 900 50  0001 C CNN
 F 1 "+BATT" H 2650 1190 50  0000 C CNN
 F 2 "" H 2650 1050 50  0001 C CNN
@@
 $EndComp
 $Comp
-L GND #PWR013
+L GND #PWR5
 U 1 1 59E51428
 P 2800 2150
-F 0 "#PWR013" H 2800 1900 50  0001 C CNN
+F 0 "#PWR5" H 2800 1900 50  0001 C CNN
 F 1 "GND" H 2800 2000 50  0001 C CNN
 F 2 "" H 2800 2150 50  0001 C CNN
@@
 $EndComp
 $Comp
-L +5V #PWR014
+L +5V #PWR12
 U 1 1 59E50C40
 P 4150 2950
-F 0 "#PWR014" H 4150 2800 50  0001 C CNN
+F 0 "#PWR12" H 4150 2800 50  0001 C CNN
 F 1 "+5V" H 4150 3090 50  0000 C CNN
 F 2 "" H 4150 2950 50  0001 C CNN
@@
 $EndComp
 $Comp
-L GND #PWR015
+L GND #PWR4
 U 1 1 59E668FA
 P 2700 3000
-F 0 "#PWR015" H 2700 2750 50  0001 C CNN
+F 0 "#PWR4" H 2700 2750 50  0001 C CNN
 F 1 "GND" H 2700 2850 50  0000 C CNN
 F 2 "" H 2700 3000 50  0001 C CNN
@@
 Connection ~ 2700 2800
 $Comp
-L GND #PWR016
+L GND #PWR6
 U 1 1 59E67A70
 P 2900 3000
-F 0 "#PWR016" H 2900 2750 50  0001 C CNN
+F 0 "#PWR6" H 2900 2750 50  0001 C CNN
 F 1 "GND" H 2900 2850 50  0000 C CNN
 F 2 "" H 2900 3000 50  0001 C CNN
@@
 	1900 2600 2050 2600
 Connection ~ 2000 2600
+$Comp
+L CONN_01X02 P2
+U 1 1 59E765D9
+P 3800 3400
+F 0 "P2" H 3800 3550 50  0000 C CNN
+F 1 "UART_TTL" V 3900 3400 50  0000 C CNN
+F 2 "Pin_Headers:Pin_Header_Straight_1x02_Pitch2.54mm" H 3800 3400 50  0001 C CNN
+F 3 "" H 3800 3400 50  0000 C CNN
+	1    3800 3400
+	0    1    1    0
+$EndComp
+Wire Wire Line
+	3750 3200 3750 2700
+Connection ~ 3750 2700
+Wire Wire Line
+	3850 3200 3850 2400
+Connection ~ 3850 2400
+$Comp
+L fiducial U3
+U 1 1 59E769F4
+P 6700 1150
+F 0 "U3" H 6500 1400 60  0001 C CNN
+F 1 "fiducial" H 6900 1350 60  0000 C CNN
+F 2 "Fiducials:Fiducial_1mm_Dia_2.54mm_Outer_CopperBottom" H 6700 1150 60  0001 C CNN
+F 3 "" H 6700 1150 60  0001 C CNN
+	1    6700 1150
+	1    0    0    -1
+$EndComp
 $EndSCHEMATC

Commit message: footprint update
Parts:
- U2: value MCP2003B -> MCP2003B-E/SN; 1st Disrtib Link https://octopart.com/search?q=MCP2003B -> https://octopart.com/mcp2003b-e%2Fsn-microchip-67312985
Changed lines of the file:
@@
 P 3250 2550
 F 0 "U2" H 3050 2850 60  0000 C CNN
-F 1 "MCP2003B" H 3350 2250 60  0000 C CNN
+F 1 "MCP2003B-E/SN" H 3150 2250 60  0000 C CNN
 F 2 "Housings_SOIC:SO-8_5.3x6.2mm_Pitch1.27mm" H 3000 2350 60  0001 C CNN
 F 3 "" H 3000 2350 60  0001 C CNN
-F 4 "https://octopart.com/search?q=MCP2003B" H 3250 2550 60  0001 C CNN "1st Disrtib Link"
+F 4 "https://octopart.com/mcp2003b-e%2Fsn-microchip-67312985" H 3250 2550 60  0001 C CNN "1st Disrtib Link"
 	1    3250 2550
 	-1   0    0    1
