File: uCLUCE_PCB.sch (KiCad schematic (older format))
At the start: 19 parts, among them J1 Screw_Terminal_01x03, J2 GS2, P1 USB_A, P2 UART_TTL, U1 PIC16F1455-I/ST, U2 MCP2003B-E/SN, U3 fiducial

Commit message: Analog sw
Parts:
- removed J2: GS2, Connectors:GS2, symbol GS2
- added U4: DG468, uCLUCE_PCB:TSOP6, symbol DG468
Connections:
- net +BATT: now also U4.5 (V+)
- net GND: now also U4.2 (V-), U4.4 (GND)
- net at C4.1, J1.2 (Pin_2), U2.6 (LBB): now also U4.1 (NO)
- net at U1.2 (RA5): now also U4.3 (IN)
- net at R1.2: now also U4.6 (COM)
Other:
- moved on the sheet: D1, R1
Changed lines of the file:
@@
 $EndComp
 $Comp
-L GND #PWR01
+L GND #PWR19
 U 1 1 59E21FB8
 P 7350 2150
-F 0 "#PWR01" H 7350 1900 50  0001 C CNN
+F 0 "#PWR19" H 7350 1900 50  0001 C CNN
 F 1 "GND" H 7350 2000 50  0000 C CNN
 F 2 "" H 7350 2150 50  0001 C CNN
@@
 $EndComp
 $Comp
-L +5V #PWR02
+L +5V #PWR17
 U 1 1 59E220C9
 P 6950 2900
-F 0 "#PWR02" H 6950 2750 50  0001 C CNN
+F 0 "#PWR17" H 6950 2750 50  0001 C CNN
 F 1 "+5V" H 6950 3040 50  0000 C CNN
 F 2 "" H 6950 2900 50  0001 C CNN
@@
 $EndComp
 $Comp
-L +5V #PWR03
+L +5V #PWR15
 U 1 1 59E2213F
 P 4050 2000
-F 0 "#PWR03" H 4050 1850 50  0001 C CNN
+F 0 "#PWR15" H 4050 1850 50  0001 C CNN
 F 1 "+5V" H 4050 2140 50  0000 C CNN
 F 2 "" H 4050 2000 50  0001 C CNN
@@
 $EndComp
 $Comp
-L +BATT #PWR04
+L +BATT #PWR3
 U 1 1 59E22154
 P 2000 2200
-F 0 "#PWR04" H 2000 2050 50  0001 C CNN
+F 0 "#PWR3" H 2000 2050 50  0001 C CNN
 F 1 "+BATT" V 1950 2400 50  0000 C CNN
 F 2 "" H 2000 2200 50  0001 C CNN
@@
 $EndComp
 $Comp
-L GND #PWR05
+L GND #PWR4
 U 1 1 59E22180
 P 2400 2200
-F 0 "#PWR05" H 2400 1950 50  0001 C CNN
+F 0 "#PWR4" H 2400 1950 50  0001 C CNN
 F 1 "GND" V 2300 2100 50  0000 C CNN
 F 2 "" H 2400 2200 50  0001 C CNN
@@
 $EndComp
 $Comp
-L GND #PWR06
+L GND #PWR18
 U 1 1 59E230A7
 P 7050 2600
-F 0 "#PWR06" H 7050 2350 50  0001 C CNN
+F 0 "#PWR18" H 7050 2350 50  0001 C CNN
 F 1 "GND" V 7000 2400 50  0001 C CNN
 F 2 "" H 7050 2600 50  0001 C CNN
@@
 MCLR
 $Comp
-L +5V #PWR07
+L +5V #PWR16
 U 1 1 59E237FB
 P 6550 2300
-F 0 "#PWR07" H 6550 2150 50  0001 C CNN
+F 0 "#PWR16" H 6550 2150 50  0001 C CNN
 F 1 "+5V" H 6550 2440 50  0000 C CNN
 F 2 "" H 6550 2300 50  0001 C CNN
@@
 $EndComp
 $Comp
-L +5V #PWR08
+L +5V #PWR9
 U 1 1 59E2335A
 P 3450 1750
-F 0 "#PWR08" H 3450 1600 50  0001 C CNN
+F 0 "#PWR9" H 3450 1600 50  0001 C CNN
 F 1 "+5V" H 3450 1890 50  0000 C CNN
 F 2 "" H 3450 1750 50  0001 C CNN
@@
 $EndComp
 $Comp
-L GND #PWR09
+L GND #PWR10
 U 1 1 59E2337A
 P 3450 1950
-F 0 "#PWR09" H 3450 1700 50  0001 C CNN
+F 0 "#PWR10" H 3450 1700 50  0001 C CNN
 F 1 "GND" H 3450 1800 50  0001 C CNN
 F 2 "" H 3450 1950 50  0001 C CNN
@@
 $EndComp
 $Comp
-L +5V #PWR010
+L +5V #PWR13
 U 1 1 59E233BF
 P 3750 1750
-F 0 "#PWR010" H 3750 1600 50  0001 C CNN
+F 0 "#PWR13" H 3750 1600 50  0001 C CNN
 F 1 "+5V" H 3750 1890 50  0000 C CNN
 F 2 "" H 3750 1750 50  0001 C CNN
@@
 $EndComp
 $Comp
-L GND #PWR011
+L GND #PWR14
 U 1 1 59E23423
 P 3750 1950
-F 0 "#PWR011" H 3750 1700 50  0001 C CNN
+F 0 "#PWR14" H 3750 1700 50  0001 C CNN
 F 1 "GND" H 3750 1800 50  0001 C CNN
 F 2 "" H 3750 1950 50  0001 C CNN
@@
 L R_Small R1
 U 1 1 59E23574
-P 2650 1450
-F 0 "R1" H 2700 1500 50  0000 L CNN
-F 1 "1k" H 2700 1400 50  0000 L CNN
-F 2 "Resistors_SMD:R_0603" H 2650 1450 50  0001 C CNN
-F 3 "" H 2650 1450 50  0001 C CNN
-F 4 "https://www.maritex.com.pl/elementy_pasywne/rezystory/rezystory_smd/rezystory_smd_0603/rezystory_smd_w_rozmiarze_0603_w_tolerancji_5/rmc0603-1k0-s.html" H 2650 1450 60  0001 C CNN "1st Disrtib Link"
-	1    2650 1450
-	1    0    0    -1
-$EndComp
-$Comp
-L +BATT #PWR012
+P 1750 1550
+F 0 "R1" V 1650 1500 50  0000 L CNN
+F 1 "1k" V 1550 1550 50  0000 L CNN
+F 2 "Resistors_SMD:R_0603" H 1750 1550 50  0001 C CNN
+F 3 "" H 1750 1550 50  0001 C CNN
+F 4 "https://www.maritex.com.pl/elementy_pasywne/rezystory/rezystory_smd/rezystory_smd_0603/rezystory_smd_w_rozmiarze_0603_w_tolerancji_5/rmc0603-1k0-s.html" H 1750 1550 60  0001 C CNN "1st Disrtib Link"
+	1    1750 1550
+	0    -1   -1   0
+$EndComp
+$Comp
+L +BATT #PWR1
 U 1 1 59E23A89
-P 2650 1050
-F 0 "#PWR012" H 2650 900 50  0001 C CNN
-F 1 "+BATT" H 2650 1190 50  0000 C CNN
-F 2 "" H 2650 1050 50  0001 C CNN
-F 3 "" H 2650 1050 50  0001 C CNN
-	1    2650 1050
-	1    0    0    -1
-$EndComp
-$Comp
-L GS2 J2
-U 1 1 59E23BFA
-P 2650 1750
-F 0 "J2" H 2750 1900 50  0000 C CNN
-F 1 "GS2" H 2750 1601 50  0001 C CNN
-F 2 "Connectors:GS2" V 2724 1750 50  0001 C CNN
-F 3 "" H 2650 1750 50  0001 C CNN
-	1    2650 1750
-	1    0    0    -1
+P 1350 1550
+F 0 "#PWR1" H 1350 1400 50  0001 C CNN
+F 1 "+BATT" H 1350 1690 50  0000 C CNN
+F 2 "" H 1350 1550 50  0001 C CNN
+F 3 "" H 1350 1550 50  0001 C CNN
+	1    1350 1550
+	0    -1   -1   0
 $EndComp
 $Comp
@@
 $EndComp
 $Comp
-L GND #PWR013
+L GND #PWR7
 U 1 1 59E51428
 P 2800 2150
-F 0 "#PWR013" H 2800 1900 50  0001 C CNN
+F 0 "#PWR7" H 2800 1900 50  0001 C CNN
 F 1 "GND" H 2800 2000 50  0001 C CNN
 F 2 "" H 2800 2150 50  0001 C CNN
@@
 $EndComp
 $Comp
-L +5V #PWR014
+L +5V #PWR11
 U 1 1 59E50C40
 P 3550 2950
-F 0 "#PWR014" H 3550 2800 50  0001 C CNN
+F 0 "#PWR11" H 3550 2800 50  0001 C CNN
 F 1 "+5V" V 3500 3150 50  0000 C CNN
 F 2 "" H 3550 2950 50  0001 C CNN
@@
 L D D1
 U 1 1 59E6633A
-P 2650 1200
-F 0 "D1" H 2650 1300 50  0000 C CNN
-F 1 "SMBD914E6327HTSA1" H 2650 1100 50  0001 C CNN
-F 2 "Diodes_SMD:D_SOT-23_ANK" H 2650 1200 50  0001 C CNN
-F 3 "" H 2650 1200 50  0000 C CNN
-F 4 "https://www.tme.eu/pl/details/smbd914e6327htsa1/diody-uniwersalne-smd/infineon-technologies/" H 2650 1200 60  0001 C CNN "1st Disrtib Link"
-	1    2650 1200
-	0    -1   -1   0
-$EndComp
-$Comp
-L GND #PWR015
+P 1500 1550
+F 0 "D1" H 1500 1650 50  0000 C CNN
+F 1 "SMBD914E6327HTSA1" H 1500 1450 50  0001 C CNN
+F 2 "Diodes_SMD:D_SOT-23_ANK" H 1500 1550 50  0001 C CNN
+F 3 "" H 1500 1550 50  0000 C CNN
+F 4 "https://www.tme.eu/pl/details/smbd914e6327htsa1/diody-uniwersalne-smd/infineon-technologies/" H 1500 1550 60  0001 C CNN "1st Disrtib Link"
+	1    1500 1550
+	-1   0    0    1
+$EndComp
+$Comp
+L GND #PWR6
 U 1 1 59E668FA
 P 2700 3000
-F 0 "#PWR015" H 2700 2750 50  0001 C CNN
+F 0 "#PWR6" H 2700 2750 50  0001 C CNN
 F 1 "GND" H 2700 2850 50  0000 C CNN
 F 2 "" H 2700 3000 50  0001 C CNN
@@
 $EndComp
 $Comp
-L GND #PWR016
+L GND #PWR8
 U 1 1 59E67A70
 P 2900 3000
-F 0 "#PWR016" H 2900 2750 50  0001 C CNN
+F 0 "#PWR8" H 2900 2750 50  0001 C CNN
 F 1 "GND" H 2900 2850 50  0000 C CNN
 F 2 "" H 2900 3000 50  0001 C CNN
@@
 $EndComp
 $Comp
-L GND #PWR017
+L GND #PWR12
 U 1 1 59E7D0F4
 P 3650 3200
-F 0 "#PWR017" H 3650 2950 50  0001 C CNN
+F 0 "#PWR12" H 3650 2950 50  0001 C CNN
 F 1 "GND" H 3650 3050 50  0000 C CNN
 F 2 "" H 3650 3200 50  0001 C CNN
@@
 Connection ~ 2700 2800
 Wire Wire Line
-	2650 1950 2650 2500
+	2650 1550 2650 2500
 Wire Wire Line
 	2800 1950 2650 1950
@@
 	3850 2500 4050 2500
 Connection ~ 3850 2500
+$Comp
+L DG468 U4
+U 1 1 5A316E90
+P 2250 1450
+F 0 "U4" H 2450 1200 60  0000 C CNN
+F 1 "DG468" H 2100 1700 60  0000 C CNN
+F 2 "uCLUCE_PCB:TSOP6" H 2250 1850 60  0001 C CNN
+F 3 "" H 2250 1850 60  0001 C CNN
+	1    2250 1450
+	-1   0    0    1
+$EndComp
+$Comp
+L GND #PWR2
+U 1 1 5A317332
+P 1850 1350
+F 0 "#PWR2" H 1850 1100 50  0001 C CNN
+F 1 "GND" V 1750 1250 50  0000 C CNN
+F 2 "" H 1850 1350 50  0001 C CNN
+F 3 "" H 1850 1350 50  0001 C CNN
+	1    1850 1350
+	0    1    1    0
+$EndComp
+Wire Wire Line
+	2650 1350 3100 1350
+Wire Wire Line
+	3100 1350 3100 2100
+Wire Wire Line
+	3100 2100 4050 2100
+$Comp
+L GND #PWR5
+U 1 1 5A31776A
+P 2650 1450
+F 0 "#PWR5" H 2650 1200 50  0001 C CNN
+F 1 "GND" V 2550 1350 50  0000 C CNN
+F 2 "" H 2650 1450 50  0001 C CNN
+F 3 "" H 2650 1450 50  0001 C CNN
+	1    2650 1450
+	0    -1   -1   0
+$EndComp
+Wire Wire Line
+	1850 1450 1350 1450
+Wire Wire Line
+	1350 1450 1350 1550
+Connection ~ 1350 1550
 $EndSCHEMATC
